File: Robots/Weeder/Chassis/Cirrus_Logic_Motor_Driver/HW/Cirrus_Logic_Motor_Driver_Tester_Ard_Shield/Cirrus_Logic_Motor_Driver_Tester_Ard_Shield.kicad_pcb (KiCad board)
At the start: 2 copper layers, 1 part

Commit message: pcb done
Parts:
- added CON1: 2x10 2.54mm male IDC header, Connector_IDC:IDC-Header_2x10_P2.54mm_Vertical, F.Cu at (109.2, 91.4)
- added J1: 1x5 2.54mm female, Connector_PinSocket_2.54mm:PinSocket_1x05_P2.54mm_Vertical, F.Cu at (38.0, 78.7)
- added J2: 1x5 2.54mm female, Connector_PinSocket_2.54mm:PinSocket_1x05_P2.54mm_Vertical, F.Cu at (30.5, 73.7)
- added J3: Screw_Terminal_01x04, TerminalBlock:TerminalBlock_bornier-4_P5.08mm, F.Cu at (30.5, 30.5)
- added Q1: IRF9Z34N, Package_TO_SOT_THT:TO-220-3_Vertical, F.Cu at (78.7, 43.2)
- added Q2: IRLZ34N, Package_TO_SOT_THT:TO-220-3_Vertical, F.Cu at (71.1, 43.2)
- added Q3: 2N7000, Package_TO_SOT_THT:TO-92_Inline_Wide, F.Cu at (94.0, 38.1)
- added Q4: IRF9Z34N, Package_TO_SOT_THT:TO-220-3_Vertical, F.Cu at (48.3, 48.3)
- added Q5: IRLZ34N, Package_TO_SOT_THT:TO-220-3_Vertical, F.Cu at (40.6, 48.3)
- added Q6: 2N7000, Package_TO_SOT_THT:TO-92_Inline_Wide, F.Cu at (63.5, 43.2)
- added R1: 220, For_Rasterboard:R_Axial_DIN0207_L6.3mm_D2.5mm_P7.62mm_Horizontal, F.Cu at (81.3, 43.2)
- added R2: 470, For_Rasterboard:R_Axial_DIN0207_L6.3mm_D2.5mm_Pinf_Horizontal, F.Cu at (81.3, 40.4)
- added R3: 220, For_Rasterboard:R_Axial_DIN0207_L6.3mm_D2.5mm_P7.62mm_Horizontal, F.Cu at (50.8, 48.3)
- added R4: 470, For_Rasterboard:R_Axial_DIN0207_L6.3mm_D2.5mm_Pinf_Horizontal, F.Cu at (50.8, 45.8)
- moved A1 91.8 mm to (45.7, 94.0), turned to 90 degrees
Connections:
- A1 pad 17: unconnected-(A1-D2-Pad17) -> /U_SSD_L
- A1 pad 18: unconnected-(A1-D3-Pad18) -> /U_SSD_H
- A1 pad 19: unconnected-(A1-D4-Pad19) -> /V_SSD_L
- A1 pad 20: unconnected-(A1-D5-Pad20) -> /V_SSD_H
- A1 pad 23: /UH -> /WL
- A1 pad 24: /UL -> /WH
- A1 pad 25: /VH -> /VL
- A1 pad 26: /VL -> /VH
- A1 pad 27: /WH -> /UL
- A1 pad 28: /WL -> /UH
- A1 pad 7: unconnected-(A1-GND-Pad7) -> GND
Routing:
- net GND: track 0.00 -> 172.7 mm, vias 0 -> 8
- net +5V: track 0.00 -> 144.8 mm, vias 0 -> 8
- net +24V: track 0.00 -> 106.6 mm, vias 0 -> 6
- net /V_SSD_L: track 0.00 -> 73.7 mm, vias 0 -> 4
- net /V_SSD_H: track 0.00 -> 55.9 mm, vias 0 -> 2
- net /U_COLD: track 0.00 -> 48.3 mm
- net /U_SSD_L: track 0.00 -> 43.2 mm, vias 0 -> 2
- net GND1: track 0.00 -> 40.6 mm
- net /U_SSD_H: track 0.00 -> 30.5 mm, vias 0 -> 2
- net /V_COLD: track 0.00 -> 17.8 mm
- net /B1: track 0.00 -> 15.2 mm
- net /A1: track 0.00 -> 15.2 mm
- net /~{EN}: track 0.00 -> 12.7 mm
- net /WL: track 0.00 -> 12.7 mm
- net /WH: track 0.00 -> 12.7 mm
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